Commit message: Add files via upload

File: agv_description/urdf/agv.xacro (robot description, xacro)
@@ -25,10 +25,10 @@
   <property name="base_depth" value="0.54" />
   <property name="base_heigth" value="0.1" />
-  <property name="base_mass" value="20" /> <!-- in kg-->
+  <property name="base_mass" value="1.8" /> <!-- in kg-->
  <!-- caster wheel radius and height -->
   <!-- caster wheel mass -->
   <property name="caster_f_height" value="0.04" />
   <property name="caster_f_radius" value="0.018" />
-  <property name="caster_f_mass" value="0.5" /> <!-- in kg-->
+  <property name="caster_f_mass" value="0.4" /> <!-- in kg-->
   <!-- caster wheel radius and height -->
   <!-- caster wheel mass -->
@@ -38,6 +38,6 @@
   <!-- Wheels -->
   <property name="wheel_mass" value="2.5" /> --> <!-- in kg-->
-  <property name="base_x_origin_to_wheel_origin" value="(0.59)" />
-  <property name="base_y_origin_to_wheel_origin" value="(0.59)" />
+  <property name="base_x_origin_to_wheel_origin" value="(0.515)" />
+  <property name="base_y_origin_to_wheel_origin" value="(0.515)" />
   <property name="base_z_origin_to_wheel_origin" value="0.0" />
  <!-- Macro for calculating inertia of cylinder -->
@@ -83,19 +83,21 @@
     <inertial>
       <mass value="${base_mass}" />
-      <origin xyz="0 0 0" />
+      <origin xyz="0 0 0" rpy="0 0 0"/>
       <!--The 3x3 rotational inertia matrix. -->
-        <box_inertia  m="${base_mass}" w="${base_width}" d="${base_depth}" h="${base_heigth}"/>
+        <inertia ixx="0.061" ixy="0.0" ixz="0.000001592"
+         iyx="0.0" iyy="0.0515" iyz="0.0"
+         izx="0.000001592" izy="0.0" izz="0.0897" />
     </inertial>
     <visual>
-      <origin xyz="0 0 0" rpy="0 0 0" />
-      <geometry>
-          <mesh filename="package://agv_description/meshes/main_assembly_stl.stl"/>
+      <origin xyz="0 0 0" rpy="${M_PI/2} 0 0" />
+      <geometry>
+          <mesh filename="package://agv_description/meshes/main_assembly.stl"/>
       </geometry>
       <material name="White" />
     </visual>
     <collision>
-      <origin xyz="0 0 0" rpy="0 0 0 " />
-      <geometry>
-          <box size="${base_width} ${base_depth} ${base_heigth}" />
+      <origin xyz="0 0 0" rpy="${M_PI/2} 0 0 " />
+      <geometry>
+          <mesh filename="package://agv_description/meshes/main_assembly.stl"/>
       </geometry>
     </collision>
@@ -103,8 +105,7 @@
   <gazebo reference="base_link">
     <material>Gazebo/White</material>
-    <turnGravityOff>false</turnGravityOff>
   </gazebo>
   <!-- Wheel Definitions -->
-  <wheel fb="front" lr="right" parent="base_link" translateX="0" translateY="0.5" flipY="1"/>
+  <wheel fb="front" lr="right" parent="base_link" translateX="0" translateY="0.5" flipY="-1"/>
   <wheel fb="front" lr="left" parent="base_link" translateX="0" translateY="-0.5" flipY="1"/>
   <!--Caster front  -->
@@ -137,5 +138,11 @@
     </joint>
   <gazebo reference="caster_front_link">
-    <turnGravityOff>false</turnGravityOff>
+    <mu1>0.1</mu1>
+    <mu2>0.1</mu2>
+    <kp>1000000.0</kp>
+    <kd>100.0</kd>
+    <minDepth>0.001</minDepth>
+    <maxVel>1.0</maxVel>
+    <material>Gazebo/Grey</material>
   </gazebo>
 <!--Caster back  -->
@@ -168,5 +175,11 @@
     </joint>
   <gazebo reference="caster_back_link">
-    <turnGravityOff>false</turnGravityOff>
+    <mu1>0.1</mu1>
+    <mu2>0.1</mu2>
+    <kp>1000000.0</kp>
+    <kd>100.0</kd>
+    <minDepth>0.001</minDepth>
+    <maxVel>1.0</maxVel>
+    <material>Gazebo/Grey</material>
   </gazebo>
   <gazebo>
@@ -184,6 +197,6 @@
       <wheelDiameter>${2*wheel_radius}</wheelDiameter>
       <broadcastTF>1</broadcastTF>
-      <wheelTorque>30</wheelTorque>
-      <wheelAcceleration>1.8</wheelAcceleration>
+      <wheelTorque>2</wheelTorque>
+      <wheelAcceleration>0.5</wheelAcceleration>
       <commandTopic>cmd_vel</commandTopic>
       <odometryFrame>odom</odometryFrame>

File: agv_description/urdf/wheel.urdf.xacro (robot description, xacro)
@@ -4,5 +4,5 @@
   <property name="wheel_radius" value="0.07" />
   <property name="wheel_height" value="0.05" />
-  <property name="wheel_mass" value="2.5" /> <!-- in kg-->
+  <property name="wheel_mass" value="0.8" /> <!-- in kg-->
   <macro name="cylinder_inertia" params="m r h">
     <inertia  ixx="${m*(3*r*r+h*h)/12}" ixy = "0" ixz = "0"
@@ -15,5 +15,5 @@
         <origin xyz="0 0 0" rpy="${flipY*M_PI/2} 0  0 " />
         <geometry>
-          <cylinder length="${wheel_height}" radius="${wheel_radius}" />
+          <mesh filename="package://agv_description/meshes/wheel.stl"/>
         </geometry>
         <material name="DarkGray" />
@@ -22,5 +22,5 @@
         <origin xyz="0 0 0" rpy="${flipY*M_PI/2} 0 0 " />
         <geometry>
-          <cylinder length="${wheel_height}" radius="${wheel_radius}" />
+          <mesh filename="package://agv_description/meshes/wheel.stl"/>
         </geometry>
       </collision>
@@ -32,11 +32,10 @@
     </link>
     <gazebo reference="${fb}_${lr}_wheel">
-      <mu1 value="1.0"/>
-      <mu2 value="1.0"/>
-      <kp  value="10000000.0" />
-      <kd  value="1.0" />
+      <mu1 value="0.1"/>
+      <mu2 value="0.1"/>
+      <kp  value="500000.0" />
+      <kd  value="10.0" />
       <fdir1 value="1 0 0"/>
       <material>Gazebo/Grey</material>
-      <turnGravityOff>false</turnGravityOff>
     </gazebo>
     <joint name="${fb}_${lr}_wheel_joint" type="continuous">
